File: Misc/Board 1/pi-crust13.brd (EAGLE design)
At the start: 101.6 x 79 mm, 28 parts, among them U1 AD9983AKSTZ_140, U2 SN54LS253_J_16, U3 SN54LS253_J_16, U4 SN54LS253_J_16

Commit message: Board Update
1.8V configured upon approval, D-Flip Flops added (choose optimal), Wire
configuration still not working correctly
Parts:
- added 100NF, 10UF: (no value), capacitor-wima:C2.5-5
- added IC1: (no value), SparkFun-PowerIC:SOT223
- added IC2: 74AC74N, 74xx-eu:DIL14
- added V1: 7474N, 74ttl-din:DIL14
- moved 3V3 5.65 mm to (98.3, 37.7)
- moved 5V 5.65 mm to (64.1, 7.26)
- moved GPIO 5.65 mm to (70.4, 16.2)
- moved I2C1 5.65 mm to (83.1, 7.26)
- moved I2C2 5.65 mm to (83.1, 2.18)
- moved SPI0 5.65 mm to (75.5, 26.3)
- moved SPI1 5.65 mm to (75.5, 21.2)
- moved UART 5.65 mm to (88.2, 37.7)
- moved GND 5.65 mm to (66.6, 2.18)
Connections:
- new net +UB: V1.14
- new net -UB: V1.7
- new net GND: IC2.7
- new net VCC: IC2.14
- net 1.8V: now also 10UF.1, IC1.2
- net 5V: now also 100NF.1, IC1.3
- net GND_WIRE: now also 100NF.2, 10UF.2, IC1.1
Routing:
- net GND_WIRE: track 0.00 -> 289.7 mm
- net 5V: track 0.00 -> 106.6 mm
- net 3V3: track 0.00 -> 98.4 mm, vias 0 -> 1
- net S1: track 0.00 -> 85.4 mm
- net 1.8V: track 0.00 -> 82.2 mm
- net R1: track 0.00 -> 74.1 mm, vias 0 -> 1
- net B6: track 0.00 -> 70.1 mm
- net S0: track 0.00 -> 67.6 mm
- net MSB2: track 0.00 -> 59.8 mm
- net MSB1: track 0.00 -> 57.4 mm
- net R2: track 0.00 -> 56.8 mm, vias 0 -> 1
- net MSB4: track 0.00 -> 53.9 mm
- net MSB3: track 0.00 -> 51.7 mm, vias 0 -> 1
- net R6: track 0.00 -> 51.3 mm, vias 0 -> 1
- net R3: track 0.00 -> 50.3 mm, vias 0 -> 1
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