File: Misc/Board 1/pi-crust14.sch (EAGLE design)
At the start: 35 parts, among them IC3 74LS595D, IC4 74LS595D, IC5 74LS595D, IC6 74LS595D, U1 AD9983AKSTZ_140, U2 SN54LS253_J_16, U3 SN54LS253_J_16, U4 SN54LS253_J_16

Commit message: Board Update 2
DFF implemented, working on and gates and binary counter
Parts:
- added IC2, IC7: 74LS595D, SparkFun-DigitalIC:74LS595D
- added IC8, IC9: 74AC11008, 74ac-logic:74AC11008
Connections:
- new net B0: IC2.G, U1.BLUE0
- new net B0_OUT: IC2.QA, U4.2C3
- new net B1: IC7.G, U1.BLUE1
- new net B1_OUT: IC7.QA, U4.1C3
- new net B2_OUT: IC6.QA, U3.2C3
- new net B3_OUT: IC5.QA, U3.1C3
- new net B6_OUT: IC2.SCL, U4.2C2
- new net B7_OUT: IC7.SCL, U4.1C2
- new net G0: IC6.RCK, U1.GREEN0
- new net G0_OUT: IC6.SCL, U3.2C2
- new net G1: IC5.RCK, U1.GREEN1
- new net G1_OUT: IC5.SCL, U3.1C2
- new net G4_OUT: IC2.QH, U4.2C1
- new net G5_OUT: IC7.QH, U4.1C1
- new net G6_OUT: IC6.QH, U3.2C1
- new net G7_OUT: IC5.QH, U3.1C1
- new net R2_0UT: IC2.QC, U4.2C0
- new net R3_OUT: IC7.QC, U4.1C0
- new net R4_OUT: IC6.QC, U3.2C0
- net 5V: now also IC2.QB, IC2.VCC, IC3.QB, IC3.VCC, IC4.QB, IC4.VCC, IC5.QB, IC5.VCC, IC6.QB, IC6.VCC, IC7.QB, IC7.VCC
- net B2: now also IC6.G; no longer U2.1C2
- net B3: now also IC5.G; no longer U2.2C2
- net B4: no longer U3.1C2
- net B4_OUT: now also U2.2C3
- net B5: no longer U3.2C2
- net B5_OUT: now also U2.1C3
- net B6: now also IC2.RCK; no longer U4.1C2
- net B7: now also IC7.RCK; no longer U4.2C2
- net CLK: now also IC2.QH*, IC5.QH*, IC6.QH*, IC7.QH*
- net G2: no longer U2.1C1
- net G2_OUT: now also U2.2C2
- net G3: no longer U2.2C1
- net G3_OUT: now also U2.1C2
- net G4: now also IC2.QF; no longer U3.1C1
- net G5: now also IC7.QF; no longer U3.2C1
- net G6: now also IC6.QF; no longer U4.1C1
- net G7: now also IC5.QF; no longer U4.2C1
- net GND_WIRE: now also IC2.GND, IC6.GND, IC7.GND, U1.EXTCLK/COAST; no longer U2.1C3, U2.2C3, U3.1C3, U3.2C3, U4.1C3, U4.2C3
- net R0_OUT: now also U2.2C1
- net R1_OUT: now also U2.1C1
- net R2: now also IC2.QE; no longer U2.1C0
- net R3: now also IC7.QE; no longer U2.2C0
- net R4: now also IC6.QE; no longer U3.1C0
- net R5: now also IC5.QE; no longer U3.2C0
- net R5_OUT: now also U3.1C0
- net R6: no longer U4.1C0
- net R6_OUT: now also U2.2C0
- net R7: no longer U4.2C0
- net R7_OUT: now also U2.1C0
Other:
- moved on the sheet: IC3, IC4, IC5, IC6

Commit message: Board Update 3
Binary Counter Added, DFF completed, Power Down Resistor added, only
thing left is to verify unused ADC pins as well as to verify all
connections are correct (add wires for RPi2 as necessary)
Parts:
- removed IC9: 74AC11008, 74ac-logic:74AC11008
- added IC10: 40193N, 40xx:40193N
- added PWRDWN_RES: 10k, rcl:R-EU_0204/7
Connections:
- new net 1: IC10G$1.QA, IC8A.I0
- new net 10K: PWRDWN_RES.1, U1.PWRDN
- new net 2: IC10G$1.QB, IC8A.I1
- new net 3: IC10G$1.QC, IC8B.I0
- new net 4: IC10G$1.QD, IC8B.I1
- new net 5: IC8A.O, IC8C.I0
- new net 6: IC8B.O, IC8C.I1
- new net DATACLK: IC10G$1.UP, U1.DATACK
- net 5V: now also IC10G$1.DOWN, IC10G$1.LOAD
- net CLK: now also IC8C.O
- net GND_WIRE: now also IC10G$1.CLEAR, PWRDWN_RES.2
Other:
- moved on the sheet: IC8A, IC8B, IC8C, IC8D
Changed lines of the file:
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@@
 <part name="IC7" library="SparkFun-DigitalIC" deviceset="74*595" device="D" technology="LS"/>
 <part name="IC8" library="74ac-logic" deviceset="74AC11008" device=""/>
-<part name="IC9" library="74ac-logic" deviceset="74AC11008" device=""/>
+<part name="IC10" library="40xx" deviceset="40193" device="N"/>
+<part name="PWRDWN_RES" library="rcl" deviceset="R-EU_" device="0204/7" value="10k"/>
 </parts>
 <sheets>
@@
 <instance part="IC2" gate="A" x="320.04" y="99.06"/>
 <instance part="IC7" gate="A" x="320.04" y="137.16"/>
-<instance part="IC8" gate="A" x="370.84" y="172.72"/>
-<instance part="IC8" gate="B" x="370.84" y="160.02"/>
-<instance part="IC8" gate="C" x="370.84" y="147.32"/>
-<instance part="IC8" gate="D" x="370.84" y="134.62"/>
-<instance part="IC9" gate="A" x="370.84" y="121.92"/>
-<instance part="IC9" gate="B" x="370.84" y="109.22"/>
-<instance part="IC9" gate="C" x="370.84" y="93.98"/>
-<instance part="IC9" gate="D" x="370.84" y="81.28"/>
+<instance part="IC8" gate="A" x="322.58" y="58.42"/>
+<instance part="IC8" gate="B" x="322.58" y="45.72"/>
+<instance part="IC8" gate="C" x="322.58" y="33.02"/>
+<instance part="IC8" gate="D" x="322.58" y="20.32"/>
+<instance part="IC10" gate="G$1" x="279.4" y="48.26"/>
+<instance part="PWRDWN_RES" gate="G$1" x="7.62" y="-5.08"/>
 </instances>
 <busses>
@@
 <pinref part="IC4" gate="A" pin="QB"/>
 </segment>
+<segment>
+<wire x1="264.16" y1="38.1" x2="261.62" y2="38.1" width="0.6096" layer="91"/>
+<label x="259.08" y="38.1" size="1.778" layer="95"/>
+<pinref part="IC10" gate="G$1" pin="DOWN"/>
+</segment>
+<segment>
+<wire x1="264.16" y1="45.72" x2="261.62" y2="45.72" width="0.6096" layer="91"/>
+<label x="259.08" y="45.72" size="1.778" layer="95"/>
+<pinref part="IC10" gate="G$1" pin="LOAD"/>
+</segment>
 </net>
 <net name="GND_WIRE" class="0">
@@
 <label x="101.6" y="86.36" size="1.778" layer="95"/>
 <pinref part="U1" gate="A" pin="GND_2"/>
+<label x="22.86" y="-5.08" size="1.778" layer="95"/>
 </segment>
 <segment>
@@
 <label x="299.72" y="83.82" size="1.778" layer="95"/>
 <pinref part="IC2" gate="A" pin="GND"/>
+</segment>
+<segment>
+<wire x1="261.62" y1="35.56" x2="264.16" y2="35.56" width="0.8128" layer="91"/>
+<label x="259.08" y="33.02" size="1.778" layer="95"/>
+<pinref part="IC10" gate="G$1" pin="CLEAR"/>
+</segment>
+<segment>
+<wire x1="12.7" y1="-5.08" x2="15.24" y2="-5.08" width="0.8128" layer="91"/>
+<pinref part="PWRDWN_RES" gate="G$1" pin="2"/>
 </segment>
 </net>
@@
 <pinref part="IC2" gate="A" pin="QH*"/>
 </segment>
+<segment>
+<wire x1="330.2" y1="33.02" x2="332.74" y2="33.02" width="0.3048" layer="91"/>
+<label x="332.74" y="33.02" size="1.778" layer="95"/>
+<pinref part="IC8" gate="C" pin="O"/>
+</segment>
 </net>
 <net name="B5_OUT" class="0">
@@
 </segment>
 </net>
+<net name="DATACLK" class="0">
+<segment>
+<pinref part="U1" gate="A" pin="DATACK"/>
+<wire x1="99.06" y1="17.78" x2="101.6" y2="17.78" width="0.3048" layer="91"/>
+<label x="104.14" y="17.78" size="1.778" layer="95"/>
+</segment>
+<segment>
+<wire x1="261.62" y1="40.64" x2="264.16" y2="40.64" width="0.3048" layer="91"/>
+<label x="259.08" y="40.64" size="1.778" layer="95"/>
+<pinref part="IC10" gate="G$1" pin="UP"/>
+</segment>
+</net>
+<net name="1" class="0">
+<segment>
+<pinref part="IC10" gate="G$1" pin="QA"/>
+<wire x1="294.64" y1="58.42" x2="297.18" y2="58.42" width="0.3048" layer="91"/>
+<label x="297.18" y="58.42" size="1.778" layer="95"/>
+</segment>
+<segment>
+<wire x1="312.42" y1="60.96" x2="314.96" y2="60.96" width="0.3048" layer="91"/>
+<label x="312.42" y="60.96" size="1.778" layer="95"/>
+<pinref part="IC8" gate="A" pin="I0"/>
+</segment>
+</net>
+<net name="2" class="0">
+<segment>
+<pinref part="IC10" gate="G$1" pin="QB"/>
+<wire x1="294.64" y1="55.88" x2="297.18" y2="55.88" width="0.3048" layer="91"/>
+<label x="297.18" y="55.88" size="1.778" layer="95"/>
+</segment>
+<segment>
+<wire x1="312.42" y1="55.88" x2="314.96" y2="55.88" width="0.3048" layer="91"/>
+<label x="312.42" y="55.88" size="1.778" layer="95"/>
+<pinref part="IC8" gate="A" pin="I1"/>
+</segment>
+</net>
+<net name="3" class="0">
+<segment>
+<pinref part="IC10" gate="G$1" pin="QC"/>
+<wire x1="294.64" y1="53.34" x2="297.18" y2="53.34" width="0.3048" layer="91"/>
+<label x="297.18" y="53.34" size="1.778" layer="95"/>
+</segment>
+<segment>
+<wire x1="312.42" y1="48.26" x2="314.96" y2="48.26" width="0.3048" layer="91"/>
+<label x="312.42" y="48.26" size="1.778" layer="95"/>
+<pinref part="IC8" gate="B" pin="I0"/>
+</segment>
+</net>
+<net name="4" class="0">
+<segment>
+<pinref part="IC10" gate="G$1" pin="QD"/>
+<wire x1="294.64" y1="50.8" x2="297.18" y2="50.8" width="0.3048" layer="91"/>
+<label x="297.18" y="50.8" size="1.778" layer="95"/>
+</segment>
+<segment>
+<wire x1="312.42" y1="43.18" x2="314.96" y2="43.18" width="0.3048" layer="91"/>
+<label x="312.42" y="43.18" size="1.778" layer="95"/>
+<pinref part="IC8" gate="B" pin="I1"/>
+</segment>
+</net>
+<net name="5" class="0">
+<segment>
+<pinref part="IC8" gate="A" pin="O"/>
+<wire x1="330.2" y1="58.42" x2="332.74" y2="58.42" width="0.3048" layer="91"/>
+<label x="332.74" y="58.42" size="1.778" layer="95"/>
+</segment>
+<segment>
+<wire x1="312.42" y1="35.56" x2="314.96" y2="35.56" width="0.3048" layer="91"/>
+<label x="312.42" y="35.56" size="1.778" layer="95"/>
+<pinref part="IC8" gate="C" pin="I0"/>
+</segment>
+</net>
+<net name="6" class="0">
+<segment>
+<pinref part="IC8" gate="B" pin="O"/>
+<wire x1="330.2" y1="45.72" x2="332.74" y2="45.72" width="0.3048" layer="91"/>
+<label x="332.74" y="45.72" size="1.778" layer="95"/>
+</segment>
+<segment>
+<wire x1="312.42" y1="30.48" x2="314.96" y2="30.48" width="0.3048" layer="91"/>
+<label x="312.42" y="30.48" size="1.778" layer="95"/>
+<pinref part="IC8" gate="C" pin="I1"/>
+</segment>
+</net>
+<net name="10K" class="0">
+<segment>
+<pinref part="U1" gate="A" pin="PWRDN"/>
+<wire x1="7.62" y1="5.08" x2="5.08" y2="5.08" width="0.6096" layer="91"/>
+</segment>
+<segment>
+<wire x1="2.54" y1="-5.08" x2="0" y2="-5.08" width="0.6096" layer="91"/>
+<pinref part="PWRDWN_RES" gate="G$1" pin="1"/>
+</segment>
+</net>
