File: Misc/Board 1/pi-crust15.sch (EAGLE design)
At the start: 43 parts, among them IC10 40193N, IC2 74LS595D, IC3 74LS595D, IC4 74LS595D, IC5 74LS595D, IC6 74LS595D, IC7 74LS595D, IC8 74AC11008, U1 AD9983AKSTZ_140, U2 SN54LS253_J_16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

Commit message: Board Update 7
Rather than using the TOBU3, I have used a 1x1 pin header and used the
dimensions of RCJ-32265 (our RCA jack).  I also had to move some
resistors and capacitors around because of the order of input.  All else
remains the same as in 14
Parts:
- removed PB, PR, Y: TOBU3, con-hirschmann:TOBU3
- added 1, 2, 3, 4, 5, 6, HOOK1, HOOK2: (no value), pinhead:PINHD-1X1
- added C7: 10u, capacitor-wima:C2.5/5
- added CP: 8.2nF, capacitor-wima:C2.5/5
- added CZ: 82nF, capacitor-wima:C2.5/5
- added JP1, JP2: (no value), pinhead:PINHD-1X5
- added RZ: 1.5k, eagle-ltspice:R0204/7
Connections:
- new net CLAMP: JP2.2, U1.CLAMP
- new net EXTCLK/COAST: JP2.1, JP2.3, U1.EXTCLK/COAST
- new net FILT: CP.2, RZ.1, U1.FILT
- new net HSOUT: JP1.4, U1.HSOUT
- new net HSYNC0: JP1.3, U1.HSYNC0
- new net N$1: CZ.2, RZ.2
- new net REFHI: C7.1, U1.REFHI
- new net REFLO: C7.2, U1.REFLO
- new net SCL: I2C1.2, JP2.5, U1.SCL
- new net SDA: I2C1.1, JP2.4, U1.SDA
- new net VSOUT/A0: JP1.2, JP1.5, U1.VSOUT/A0
- new net VSYNC0: JP1.1, U1.VSYNC0
- net 1.8V: now also CP.1, CZ.1
- net GND_WIRE: now also U1.HSYNC1, U1.O/E_FIELD, U1.VSYNC1; no longer U1.EXTCLK/COAST
- net PBIN_0: now also 5.1; no longer PB.1
- net PBIN_1: now also 6.1; no longer PB.2
- net PRIN_0: now also 1.1; no longer PR.1
- net PRIN_1: now also 2.1; no longer PR.2
- net YIN_0: now also 3.1; no longer Y.1
- net YIN_1: now also 4.1; no longer Y.2
Other:
- note added: "RPI 2 Connection"
- moved on the sheet: SPI1
